File: WISP_STM32_test_board.kicad_pcb (KiCad board)
At the start: 2 copper layers, 50 x 50 mm, 30 parts, among them J1 Conn_02x05_Odd_Even, J2 Conn_02x01, J3 Conn_02x01, J5 Conn_01x02_Pin, J6 Conn_01x09_Pin, U1 MAX3072E, U2 MAX3072E, U3 AMS1117-3.3, U4 STM32F446RETx

Commit message: Full 15 rough draft
Parts:
- added R4: 10K, Resistor_SMD:R_0805_2012Metric_Pad1.20x1.40mm_HandSolder, F.Cu at (168.5, 82.2)
- added R5: 10K, Resistor_SMD:R_0805_2012Metric_Pad1.20x1.40mm_HandSolder, F.Cu at (168.5, 72.0)
- added SW1: SW_Push, Button_Switch_THT:SW_PUSH_6mm, F.Cu at (172.8, 82.5)
- added SW2: SW_Push, Button_Switch_THT:SW_PUSH_6mm, F.Cu at (172.8, 72.0)
- moved J6 13.6 mm to (179.5, 66.0), turned to 180 degrees
- moved U4 4.83 mm to (159.2, 60.7)
- moved R1 3.20 mm to (157.5, 52.5), turned to 180 degrees
- moved D3 2.24 mm to (158.0, 88.5)
- moved J5 2.12 mm to (128.0, 71.5)
- moved R3 1.80 mm to (151.5, 88.5)
- moved D1 1.41 mm to (129.0, 82.5)
- moved FB1 1.41 mm to (129.0, 87.5)
- moved R2 1.41 mm to (161.0, 83.0)
- moved J1 1.39 mm to (163.6, 48.5)
- moved C1 1.12 mm to (136.5, 87.5)
- moved C2 1.12 mm to (150.5, 82.5)
- moved D2 1.12 mm to (155.5, 83.0), turned to 180 degrees
- moved F1 1.12 mm to (137.0, 82.5)
- moved U3 1.12 mm to (144.0, 85.2)
Connections:
- J6 pad 1: /SPI3_STCP -> +3.3V
- J6 pad 2: /SPI3_SCK -> GND
- J6 pad 3: /SPI3_MOSI -> /I2C3_SDA
- J6 pad 4: /I2C1_SCL -> /I2C3_SCL
- J6 pad 6: /I2C3_SCL -> /I2C1_SCL
- J6 pad 7: /I2C3_SDA -> /SPI3_MOSI
- J6 pad 8: GND -> /SPI3_SCK
- J6 pad 9: +3.3V -> /SPI3_STCP
- U4 pad 27: unconnected-(U4-PB1-Pad27) -> /CTRL_1
- U4 pad 33: unconnected-(U4-PB12-Pad33) -> /CTRL_2
Routing:
- net +3.3V: track 0.00 -> 121.4 mm
- net /SPI3_MOSI: track 0.00 -> 36.4 mm, vias 0 -> 2
- net /USART1_RX: track 0.00 -> 32.7 mm, vias 0 -> 2
- net /USART3_TX: track 0.00 -> 32.1 mm, vias 0 -> 2
- net /USART1_TX: track 0.00 -> 31.4 mm
- net /RS485_T1: track 0.00 -> 29.6 mm
- net GND: track 0.00 -> 29.3 mm, vias 0 -> 2
- net /USART3_RX: track 0.00 -> 28.0 mm, vias 0 -> 2
- net /SPI3_STCP: track 0.00 -> 27.6 mm, vias 0 -> 2
- net /I2C1_SDA: track 0.00 -> 26.9 mm, vias 0 -> 2
- net /I2C1_SCL: track 0.00 -> 26.7 mm, vias 0 -> 2
- net /SPI3_SCK: track 0.00 -> 24.5 mm, vias 0 -> 2
- net /RS485_T3: track 0.00 -> 19.2 mm
- net Net-(U3-VI): track 0.00 -> 18.8 mm
- net /CTRL_1: track 0.00 -> 18.8 mm
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- added copper zone on B.Cu, net GND
Other:
- board size 50 x 50 mm -> 60 x 50 mm
- board text added: "3.3v"
- board text added: "GND"
- board text added: "I2C1_SCL"
- board text added: "I2C1_SDA"
- board text added: "I2C3_SCL"
- board text added: "I2C3_SDA"
- board text added: "SPI3_MOSI"
- board text added: "SPI3_SCK"
- board text added: "SPI3_STCP"

Commit message: V1 routing
Parts:
- removed J6: Conn_01x09_Pin, Connector_PinSocket_2.54mm:PinSocket_1x09_P2.54mm_Vertical
- added J4: Conn_01x10_Pin, Connector_JST:JST_XH_B10B-XH-A_1x10_P2.50mm_Vertical, F.Cu at (177.5, 70.0)
- added SW3: SW_SPST, Button_Switch_SMD:SW_DIP_SPSTx01_Slide_6.7x4.1mm_W6.73mm_P2.54mm_LowProfile_JPin, F.Cu at (127.5, 77.9)
- moved J1 8.05 mm to (155.6, 49.0)
- moved R5 5.00 mm to (168.5, 77.0)
- moved SW2 5.00 mm to (172.8, 77.0)
- moved J5 4.50 mm to (128.0, 67.0)
- moved U4 4.21 mm to (161.0, 64.5)
- moved R4 3.50 mm to (168.5, 85.8)
- moved SW1 3.50 mm to (172.8, 86.0)
- moved R1 3.16 mm to (158.5, 55.5)
- moved D1 2.55 mm to (129.5, 85.0)
- moved F1 2.55 mm to (136.5, 85.0)
- moved FB1 1.12 mm to (129.5, 88.5)
- moved C1 1.00 mm to (136.5, 88.5)
Connections:
- F1 pad 2: Net-(F1-Pad2) -> Net-(SW3-A)
- FB1 pad 1: Net-(F1-Pad2) -> Net-(SW3-B)
- U4 pad 37: unconnected-(U4-PC6-Pad37) -> /I2C_AD1
- U4 pad 40: /I2C3_SDA -> unconnected-(U4-PC9-Pad40)
- U4 pad 41: /I2C3_SCL -> unconnected-(U4-PA8-Pad41)
- U4 pad 53: unconnected-(U4-PC12-Pad53) -> /I2C_AD2
- U4 pad 9: unconnected-(U4-PC1-Pad9) -> /I2C_AD0
Routing:
- net +3.3V: track 121.4 -> 232.8 mm, vias 0 -> 7
- net GND: track 29.3 -> 110.3 mm, vias 2 -> 8
- net /CTRL_2: track 0.00 -> 25.8 mm, vias 0 -> 2
- net /I2C_AD0: track 0.00 -> 24.0 mm, vias 0 -> 2
- net /NRST: track 15.4 -> 38.8 mm
- net /I2C_AD2: track 0.00 -> 17.9 mm, vias 0 -> 2
- net /I2C3_SCL: track 15.4 -> 0.00 mm
- net Net-(SW3-A): track 0.00 -> 14.7 mm
- net /I2C3_SDA: track 14.6 -> 0.00 mm
- net /I2C_AD1: track 0.00 -> 12.4 mm
- net Net-(F1-Pad2): track 12.1 -> 0.00 mm
- net /SWO: track 9.60 -> 18.9 mm
- net /RS485_T3: track 19.2 -> 28.4 mm, vias 0 -> 2
- net /SW_TICK: track 9.80 -> 18.6 mm
- net Net-(SW3-B): track 0.00 -> 7.79 mm
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Other:
- board text removed: "3.3v"
- board text removed: "GND"
- board text removed: "I2C1_SCL"
- board text removed: "I2C1_SDA"
- board text removed: "I2C3_SCL"
- board text removed: "I2C3_SDA"
- board text removed: "SPI3_MOSI"
- board text removed: "SPI3_SCK"
- board text removed: "SPI3_STCP"

Commit message: Rough draft V2
Parts:
- removed C1, C2: 10uF, Capacitor_SMD:C_0805_2012Metric_Pad1.18x1.45mm_HandSolder
- removed D1: B5819W, Diode_SMD:D_SOD-123
- removed D3: Red, LED_SMD:LED_0805_2012Metric_Pad1.15x1.40mm_HandSolder
- removed F1: 500mA, Fuse:Fuse_0805_2012Metric_Pad1.15x1.40mm_HandSolder
- removed FB1: 100 @ 100MHz, Resistor_SMD:R_0805_2012Metric_Pad1.20x1.40mm_HandSolder
- removed R3: 2k2, Resistor_SMD:R_0805_2012Metric_Pad1.20x1.40mm_HandSolder
- removed SW3: SW_SPST, Button_Switch_SMD:SW_DIP_SPSTx01_Slide_6.7x4.1mm_W6.73mm_P2.54mm_LowProfile_JPin
- removed U3: AMS1117-3.3, Package_TO_SOT_SMD:SOT-223-3_TabPin2
- added C16: 10uF, Capacitor_SMD:C_0805_2012Metric_Pad1.18x1.45mm_HandSolder, F.Cu at (128.5, 85.0)
- added C17: 100nF, Capacitor_SMD:C_0805_2012Metric_Pad1.18x1.45mm_HandSolder, F.Cu at (144.9, 80.5)
- added C18: 22uF, Capacitor_SMD:C_0805_2012Metric_Pad1.18x1.45mm_HandSolder, F.Cu at (150.4, 84.0)
- added C19: 22uF, Capacitor_SMD:C_0805_2012Metric_Pad1.18x1.45mm_HandSolder, F.Cu at (144.9, 84.0)
- added D5: Red, LED_SMD:LED_0805_2012Metric_Pad1.15x1.40mm_HandSolder, F.Cu at (134.5, 78.5)
- added L2: 2.2uH, Inductor_SMD:L_0805_2012Metric_Pad1.05x1.20mm_HandSolder, F.Cu at (150.2, 80.5)
- added R6: 120, Resistor_SMD:R_0805_2012Metric_Pad1.20x1.40mm_HandSolder, F.Cu at (128.5, 55.0)
- added R7: 120, Resistor_SMD:R_0805_2012Metric_Pad1.20x1.40mm_HandSolder, F.Cu at (128.5, 45.0)
- added R9: 2k2, Resistor_SMD:R_0805_2012Metric_Pad1.20x1.40mm_HandSolder, F.Cu at (134.5, 83.5)
- added SW5: SW_SPST, Button_Switch_THT:SW_CK_JS202011CQN_DPDT_Straight, F.Cu at (126.7, 81.0)
- added U6: AP63203WU, Package_TO_SOT_SMD:TSOT-23-6, F.Cu at (139.5, 81.5)
- J1: footprint Connector_PinSocket_2.54mm:PinSocket_2x05_P2.54mm_Vertical -> Connector_PinHeader_2.54mm:PinHeader_2x05_P2.54mm_Vertical
- J2, J3: footprint Connector_PinSocket_2.54mm:PinSocket_1x02_P2.54mm_Vertical -> TerminalBlock:TerminalBlock_Xinya_XY308-2.54-2P_1x02_P2.54mm_Horizontal
- J4: footprint Connector_JST:JST_XH_B10B-XH-A_1x10_P2.50mm_Vertical -> Connector_PinHeader_2.54mm:PinHeader_1x10_P2.54mm_Vertical
- J5: footprint Connector_JST:JST_PH_B2B-PH-K_1x02_P2.00mm_Vertical -> Connector_PinSocket_2.54mm:PinSocket_1x02_P2.54mm_Vertical
- moved SW1 14.2 mm to (159.8, 80.2)
- moved R4 12.9 mm to (156.0, 82.5), turned to -90 degrees
- moved D2 7.52 mm to (156.0, 75.5)
- moved R2 7.52 mm to (160.5, 75.5)
- moved R5 5.70 mm to (170.0, 82.5), turned to -90 degrees
- moved SW2 3.29 mm to (173.2, 80.2)
- moved C13 2.54 mm to (134.0, 54.5)
- moved J1 2.50 mm to (155.5, 46.5)
- moved C8 1.78 mm to (144.5, 68.5)
- moved C10 1.78 mm to (148.0, 73.0)
- moved C11 1.78 mm to (151.0, 71.0)
- moved C3 1.78 mm to (137.5, 73.0)
- moved C4 1.78 mm to (141.0, 73.0)
- moved C5 1.78 mm to (144.5, 73.0)
- moved C6 1.78 mm to (137.5, 68.5)
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Routing:
- net GND: track 110.3 -> 73.8 mm, vias 8 -> 13
- net Net-(SW5-B): track 0.00 -> 23.8 mm
- net Net-(U3-VI): track 23.2 -> 0.00 mm, vias 2 -> 0
- net Net-(SW3-A): track 14.7 -> 0.00 mm
- net Net-(J2-Pin_2): track 7.40 -> 18.3 mm
- net Net-(J2-Pin_1): track 7.92 -> 17.4 mm
- net Net-(U6-BST): track 0.00 -> 9.40 mm
- net +3.3V: track 232.8 -> 224.4 mm, vias 7 -> 5
- net Net-(SW3-B): track 7.79 -> 0.00 mm
- net Net-(D2-A): track 14.8 -> 7.10 mm
- net Net-(J3-Pin_2): track 8.18 -> 15.8 mm
- net Net-(J3-Pin_1): track 7.65 -> 14.8 mm
- net Net-(U6-SW): track 0.00 -> 5.98 mm
- net /CTRL_2: track 25.8 -> 31.3 mm
- net /SPI3_MOSI: track 34.6 -> 39.3 mm
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Other:
- board size 60 x 50 mm -> 60 x 45 mm
- board text added: "+"
- board text added: "-"
- board text added: "3.3V"
- board text added: "A"
- board text added: "B"
- board text added: "DISPLAY BOARD"
- board text added: "OFF"
- board text added: "ON"
- board text added: "SENSORS"
- board text added: "ST-LINK"
- board text added: "VALVES"

Commit message: John revisions 9/7
Parts:
- removed J2, J3: Conn_02x01, TerminalBlock:TerminalBlock_Xinya_XY308-2.54-2P_1x02_P2.54mm_Horizontal
- added J6: Conn_01x03_Socket, TerminalBlock:TerminalBlock_Xinya_XY308-2.54-3P_1x03_P2.54mm_Horizontal, F.Cu at (128.2, 58.9)
- added J7: Conn_01x03_Socket, TerminalBlock:TerminalBlock_Xinya_XY308-2.54-3P_1x03_P2.54mm_Horizontal, F.Cu at (128.2, 47.5)
- moved C12 1.75 mm to (134.0, 66.2)
- moved R6 0.90 mm to (128.0, 55.8)
- moved R7 0.90 mm to (128.0, 44.2)
- moved C13 0.79 mm to (134.2, 55.2)
Routing:
- net GND: track 73.8 -> 62.1 mm, vias 13 -> 14
- net Net-(J7-Pin_2): track 14.8 -> 17.8 mm
- net Net-(J7-Pin_3): track 15.8 -> 18.9 mm
- net Net-(U2-VCC): track 2.60 -> 4.35 mm
- net +3.3V: track 224.4 -> 223.3 mm
- net Net-(U1-VCC): track 4.61 -> 5.49 mm
- net Net-(J6-Pin_3): track 18.3 -> 18.8 mm
- net Net-(C18-Pad1): vias 1 -> 0
- added copper zone on F.Cu, net GND
Other:
- board text added: "<- GND"
- board text added: "NRST"
- board text added: "SWCLK"
- board text added: "SWDIO"
- board text added: "SWO"
- board text added: "X"

Commit message: Fixed decoupling capacitors
Parts:
- moved C13 4.26 mm to (137.5, 52.5)
- moved C12 4.16 mm to (137.5, 64.0)
Connections:
- C12 pad 1: +3.3V -> GND
- C12 pad 2: Net-(U2-VCC) -> +3.3V
- C13 pad 1: +3.3V -> GND
- C13 pad 2: Net-(U1-VCC) -> +3.3V
- U1 pad 8: Net-(U1-VCC) -> +3.3V
- U2 pad 8: Net-(U2-VCC) -> +3.3V
Routing:
- net +3.3V: track 223.3 -> 233.1 mm
- net Net-(U1-VCC): track 5.49 -> 0.00 mm
- net Net-(U2-VCC): track 4.35 -> 0.00 mm

Commit message: Rough draft V3
Parts:
- added H1: MountingHole, MountingHole:MountingHole_2.2mm_M2, F.Cu at (181.5, 45.0)
- added H2: MountingHole, MountingHole:MountingHole_2.2mm_M2, F.Cu at (181.5, 85.0)
- added H3: MountingHole, MountingHole:MountingHole_2.2mm_M2, F.Cu at (126.5, 85.0)
- added H4: MountingHole, MountingHole:MountingHole_2.2mm_M2, F.Cu at (126.5, 45.0)
- added TP1: 3.3V, TestPoint:TestPoint_Pad_1.0x1.0mm, F.Cu at (172.0, 75.8)
- added TP2: GND, TestPoint:TestPoint_Pad_1.0x1.0mm, F.Cu at (176.2, 75.8)
- L2: value 2.2uH -> 4.7uH
- moved C16 15.1 mm to (143.6, 84.8)
- moved R9 13.0 mm to (131.2, 71.0), turned to -90 degrees
- moved SW5 10.3 mm to (136.2, 84.8), turned to 180 degrees
- moved C18 9.21 mm to (141.9, 80.5), turned to 90 degrees
- moved U6 6.25 mm to (145.8, 81.8)
- moved J5 4.46 mm to (126.8, 72.2)
- moved C17 4.14 mm to (148.6, 78.8)
- moved D5 4.10 mm to (131.2, 76.0), turned to -90 degrees
- moved C19 4.06 mm to (148.9, 84.8)
- moved R7 2.37 mm to (130.2, 45.0), turned to -90 degrees
- moved SW2 2.25 mm to (171.0, 80.2)
- moved J7 2.04 mm to (128.2, 49.5)
- moved R5 2.02 mm to (168.0, 82.8)
- moved R6 2.00 mm to (128.0, 57.8)
- moved J6 1.83 mm to (128.2, 60.8)
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Routing:
- net +3.3V: track 233.1 -> 248.1 mm
- net Net-(SW5-B): track 23.8 -> 13.7 mm
- net Net-(C18-Pad1): track 3.42 -> 13.1 mm, vias 0 -> 2
- net VCC: track 14.5 -> 18.4 mm
- net Net-(U6-BST): track 9.40 -> 6.07 mm
- net Net-(J7-Pin_3): track 18.9 -> 16.0 mm
- net Net-(J6-Pin_3): track 18.8 -> 16.2 mm
- net Net-(U6-SW): track 5.98 -> 8.37 mm
- net /CTRL_1: track 13.9 -> 16.2 mm
- net Net-(J6-Pin_2): track 17.7 -> 16.0 mm
- net Net-(J7-Pin_2): track 17.8 -> 16.5 mm
- net Net-(R5-Pad2): track 11.1 -> 12.3 mm
- net /SPI3_SCK: track 20.1 -> 19.4 mm
- net /I2C_AD2: track 18.6 -> 17.8 mm
- net /I2C1_SDA: track 24.0 -> 23.3 mm
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Other:
- outline, holes or cut-outs redrawn
- board text added: "-> DISPLAY BOARD"
- board text added: "GND"
- board text removed: "DISPLAY BOARD"

Commit message: Rough draft V4
Parts:
- removed C10, C7, C8, C9: 100nF, Capacitor_SMD:C_0805_2012Metric_Pad1.18x1.45mm_HandSolder
- added C1: 100nF, Capacitor_SMD:C_0603_1608Metric, F.Cu at (155.5, 71.2)
- C11, C3, C4, C5, C6: footprint Capacitor_SMD:C_0805_2012Metric_Pad1.18x1.45mm_HandSolder -> Capacitor_SMD:C_0603_1608Metric
- L2: footprint Inductor_SMD:L_0805_2012Metric_Pad1.05x1.20mm_HandSolder -> Inductor_SMD:L_Taiyo-Yuden_MD-4040
- moved C3 32.0 mm to (165.8, 60.0), turned to -90 degrees
- moved C6 24.8 mm to (161.8, 71.0), turned to 180 degrees
- moved C4 23.0 mm to (154.8, 56.0), turned to 0 degrees
- moved C5 15.2 mm to (150.8, 60.5), turned to -90 degrees
- moved R2 14.8 mm to (148.8, 66.5), turned to 90 degrees
- moved D2 8.55 mm to (148.8, 71.0), turned to -90 degrees
- moved R6 8.00 mm to (134.2, 62.8), turned to -90 degrees
- moved R7 7.85 mm to (134.2, 51.8)
- moved C13 4.35 mm to (139.2, 56.2)
- moved U1 4.35 mm to (139.2, 52.0)
- moved C12 3.05 mm to (139.2, 66.5)
- moved U2 3.05 mm to (139.2, 62.5)
- moved U4 2.93 mm to (158.2, 63.5)
- moved C11 2.72 mm to (152.2, 70.0)
- moved R1 1.90 mm to (157.8, 53.8), turned to 90 degrees
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Connections:
- C17 pad 1: Net-(U6-BST) -> Net-(U6-SW)
- C17 pad 2: Net-(U6-SW) -> Net-(U6-BST)
- L2 pad 1: Net-(U6-BST) -> Net-(U6-SW)
Routing:
- net +3.3V: track 248.1 -> 164.2 mm
- net GND: track 62.2 -> 21.5 mm, vias 53 -> 38
- net /NRST: track 40.5 -> 17.6 mm
- net /USART1_RX: track 39.9 -> 24.3 mm, vias 2 -> 4
- net /CTRL_2: track 30.6 -> 19.4 mm
- net /RS485_T1: track 34.8 -> 24.1 mm, vias 0 -> 2
- net /RS485_T3: track 28.4 -> 18.8 mm, vias 2 -> 0
- net /I2C1_SCL: track 29.7 -> 21.8 mm, vias 2 -> 0
- net Net-(J7-Pin_2): track 16.5 -> 9.31 mm
- net /SPI3_MOSI: track 40.0 -> 32.9 mm, vias 0 -> 3
- net Net-(J7-Pin_3): track 16.0 -> 9.33 mm
- net Net-(J6-Pin_3): track 16.2 -> 9.64 mm
- net Net-(J6-Pin_2): track 16.0 -> 9.62 mm
- net /USART1_TX: track 29.0 -> 23.2 mm, vias 0 -> 2
- net /SPI3_SCK: track 19.4 -> 24.9 mm
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