File: WISP_STM32_test_board.kicad_pcb (KiCad board)
At the start: 2 copper layers, 60 x 45 mm, 40 parts, among them J1 Conn_02x05_Odd_Even, J4 Conn_01x10_Pin, J5 Conn_01x02_Pin, J6 Conn_01x03_Socket, J7 Conn_01x03_Socket, SW1 SW_Push, SW2 SW_Push, SW5 SW_SPST, U1 MAX3072E, U2 MAX3072E, U4 STM32F446RETx, U6 AP63203WU

Commit message: New MCU STM32F401
Parts:
- removed D2: Green, LED_SMD:LED_0805_2012Metric_Pad1.15x1.40mm_HandSolder
- removed R2: 2k2, Resistor_SMD:R_0805_2012Metric_Pad1.20x1.40mm_HandSolder
- removed U4: STM32F446RETx, Package_QFP:LQFP-64_10x10mm_P0.5mm
- added C2: 100nF, Capacitor_SMD:C_0603_1608Metric, F.Cu at (150.3, 66.8)
- added D1: Green, LED_SMD:LED_0805_2012Metric_Pad1.15x1.40mm_HandSolder, F.Cu at (147.5, 72.8)
- added R3: 2k2, Resistor_SMD:R_0805_2012Metric_Pad1.20x1.40mm_HandSolder, F.Cu at (147.5, 68.1)
- added U3: STM32F401RCTx, Package_QFP:LQFP-64_10x10mm_P0.5mm, F.Cu at (158.3, 63.5)
- TP1, TP2: footprint TestPoint:TestPoint_Pad_1.0x1.0mm -> Custom_Components:TestPoint_Pad_1.0x1.0mm_CUSTOM
Connections:
- U1 pad 1: /USART3_RX -> /USART2_RX
- U1 pad 4: /USART3_TX -> /USART2_TX
Routing:
- net /USART2_TX: track 0.00 -> 37.3 mm, vias 0 -> 2
- net /USART3_TX: track 33.8 -> 0.00 mm, vias 2 -> 0
- net /USART2_RX: track 0.00 -> 31.4 mm, vias 0 -> 2
- net /USART3_RX: track 28.9 -> 0.00 mm, vias 2 -> 0
- net Net-(D1-A): track 0.00 -> 14.4 mm, vias 0 -> 2
- net Net-(D2-A): track 10.6 -> 0.00 mm
- net +3.3V: track 164.2 -> 171.1 mm
- net GND: track 21.5 -> 24.6 mm, vias 38 -> 41
- net Net-(D1-K): track 0.00 -> 2.74 mm
- net Net-(D2-K): track 2.48 -> 0.00 mm
- net /SPI3_MOSI: track 32.9 -> 31.0 mm
- net /SPI3_SCK: track 24.9 -> 25.8 mm
- net /SW_TICK: track 19.4 -> 19.9 mm
Other:
- board text added: "-> DISPLAY"
- board text added: "CLK"
- board text added: "IO"
- board text removed: "-> DISPLAY BOARD"
- board text removed: "SWCLK"
- board text removed: "SWDIO"
