File: WISP_STM32_test_board.kicad_sch (KiCad schematic)
At the start: 40 parts, among them J1 Conn_02x05_Odd_Even, J4 Conn_01x10_Pin, J5 Conn_01x02_Pin, J6 Conn_01x03_Socket, J7 Conn_01x03_Socket, SW1 SW_Push, SW2 SW_Push, SW5 SW_SPST, U1 MAX3072E, U2 MAX3072E, U4 STM32F446RETx, U6 AP63203WU

Commit message: New MCU STM32F401
Parts:
- removed D2: Green, LED_SMD:LED_0805_2012Metric_Pad1.15x1.40mm_HandSolder, symbol Device:LED_Small
- removed R2: 2k2, Resistor_SMD:R_0805_2012Metric_Pad1.20x1.40mm_HandSolder, symbol Device:R
- removed U4: STM32F446RETx, Package_QFP:LQFP-64_10x10mm_P0.5mm, symbol MCU_ST_STM32F4:STM32F446RETx
- added C2: 100nF, Capacitor_SMD:C_0603_1608Metric, symbol Device:C
- added D1: Green, LED_SMD:LED_0805_2012Metric_Pad1.15x1.40mm_HandSolder, symbol Device:LED_Small
- added R3: 2k2, Resistor_SMD:R_0805_2012Metric_Pad1.20x1.40mm_HandSolder, symbol Device:R
- added U4: STM32F401RCTx, Package_QFP:LQFP-64_10x10mm_P0.5mm, symbol MCU_ST_STM32F4:STM32F401RCTx
- TP1, TP2: footprint TestPoint:TestPoint_Pad_1.0x1.0mm -> Custom_Components:TestPoint_Pad_1.0x1.0mm_CUSTOM
Connections:
- net +3.3V: now also C2.1, U4.1 (VBAT), U4.13 (VREF+), U4.19 (VDD), U4.32 (VDD), U4.48 (VDD), U4.64 (VDD)
- net BOOT0: now also U4.60 (BOOT0)
- net CTRL_1: now also U4.27 (PB1)
- net CTRL_2: now also U4.33 (PB12)
- net GND: now also C2.2, R3.2, U4.12 (VSSA), U4.18 (VSS), U4.31 (VSS), U4.47 (VSS), U4.63 (VSS)
- net I2C1_SCL: now also U4.58 (PB6)
- net I2C1_SDA: now also U4.59 (PB7)
- net I2C_AD0: now also U4.9 (PC1)
- net I2C_AD1: now also U4.37 (PC6)
- net I2C_AD2: now also U4.52 (PC11)
- net NRST: now also U4.7 (NRST)
- net RS485_T1: now also U4.38 (PC7)
- net RS485_T3: now also U4.8 (PC0)
- net SPI3_MOSI: now also U4.53 (PC12)
- net SPI3_SCK: now also U4.51 (PC10)
- net SPI3_STCP: now also U4.57 (PB5)
- net SWO: now also U4.55 (PB3)
- net SW_TICK: now also U4.49 (PA14)
- net SW_TMS: now also U4.46 (PA13)
- net USART1_RX: now also U4.43 (PA10)
- net USART1_TX: now also U4.42 (PA9)
- net USART3_RX renamed USART2_RX
- net USART2_RX: now also U4.17 (PA3)
- net USART3_TX renamed USART2_TX
- net USART2_TX: now also U4.16 (PA2)
- new net: D1.2 (A), U4.21 (PA5)
- new net: D1.1 (K), R3.1
- no-connect marks 33 -> 32
Other:
- moved on the sheet: R1
